File: KiCad Scheme/SoundNode/SoundNode.kicad_sch (KiCad schematic)
At the start: 0 parts

Commit message: KiCad Scheme, README.md Power consumption and notes sections
Parts:
- added BT1, BT2: Li-Ion Cell, symbol Device:Battery_Cell
- added C1: 40n, PCM_SparkFun-Capacitor:C_0603_1608Metric, symbol PCM_SparkFun-Capacitor:C
- added LS1: Speaker 4R, symbol Device:Speaker
- added Q1: NMOS, symbol Simulation_SPICE:NMOS
- added R1: 270k, symbol Device:R
- added R2, R6: 100k, symbol Device:R
- added R3: 4K53, symbol Device:R
- added R4: 7K5, symbol Device:R
- added R5: 22R, symbol Device:R
- added TH1: 100K B4100/B3950 NTC, symbol Device:Thermistor_NTC
- added U1: ESP32-C3-SuperMini, symbol CustomModules:ESP32-C3-SuperMini
- added U2: MAX98357A, symbol CustomModules:MAX98357A-Module
- added U3: 2S BMS, symbol CustomModules:2S-BMS-LiIon
- added U4, U5: Mini560, symbol CustomModules:Mini560
- added U6: IP2326, symbol CustomModules:IP2326-Module
Connections:
- new net: R4.1, U5. (En)
- new net: R4.2, U5. (En)
- new net: U1. (0), U4. (En)
- new net: R3.1, U4. (En)
- new net: R3.2, U4. (En)
- new net: BT1.1 (+), U3. (0V)
- new net: BT1.2 (-), BT2.1 (+), U3. (0V), U6. (B-)
- new net: LS1.1, U2. (VIN)
- new net: LS1.2, U2. (VIN)
- new net: Q1.1 (D), U5. (En)
- new net: TH1.1, U6. (B-)
- new net: TH1.2, U6. (B-)
- new net: C1.1, R1.2, R2.1, U1. (0)
- new net: Q1.2 (G), R5.2, R6.2
- new net: U1. (0), U2. (VIN) (x3)
- new net: BT2.2 (-), U3. (0V)
- new net: R5.1, U1. (0)
- new net GND: C1.2, Q1.3 (S), R2.2, R6.1, U1. (0), U2. (VIN), U3. (0V), U4. (En), U5. (En), U6. (B-)
- new net VRAW: R1.1, U3. (0V), U4. (En), U5. (En), U6. (B-)
- no-connect marks 0 -> 15

Commit message: Schematic images, Update README.md
Connections:
- new net: U1. (0), U4. (En)
- new net: U1. (0), U2. (VIN) (x3)
Other:
- title: (none) -> Wi-Fi Sound Node
Changed lines of the file:
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@@
 	(generator_version "9.0")
 	(paper "A4")
+	(title_block
+		(title "Wi-Fi Sound Node")
+		(date "2026-02-10")
+		(rev "1.0")
+		(comment 1 "Author: Kiryl Alishkevich")
+	)
 	(text_box "R3 (4.53 kΩ) sets Mini560 output voltage to ≈3.3 V"
 		(exclude_from_sim no)
